Commit message: modified main and gazebo modules of XACRO and created launch file to spawn two box_bots that each have their own topics i.e. box_bot1/odom

File: my_box_bot_description/urdf/box_bot.gazebo.xacro (robot description, xacro)
@@ -1,4 +1,5 @@
 <?xml version="1.0"?>
 <robot xmlns:xacro="http://www.ros.org/wiki/xacro">
+<xacro:arg name="robot_name" default="box_bot" />
 <xacro:macro name="gazebo_elements">
   <gazebo reference="left_wheel">
@@ -42,4 +43,4 @@
     <material>Gazebo/Red</material>
   </gazebo>
-    </xacro:macro>
+  </xacro:macro>
 </robot>

File: my_box_bot_description/urdf/box_bot.xacro (robot description, xacro)
@@ -1,4 +1,5 @@
 <?xml version="1.0"?>
 <robot xmlns:xacro="http://www.ros.org/wiki/xacro" name="my_box_bot">
+<xacro:property name="robot_name" value="$(arg robot_name)"/>
 <xacro:include filename="$(find my_box_bot_description)/urdf/box_bot.gazebo.xacro" />
 <xacro:property name="body_width" value="0.1"/>
@@ -202,5 +203,4 @@
       </inertial>
   </link>
-Exercise
   <joint name="back_roll_joint" type="continuous">
     <origin rpy="0 0 0" xyz="0 0 0" />
@@ -238,3 +238,44 @@
     <dynamics damping="0.0" friction="0.1"/>
   </joint>
+    <gazebo>
+    <plugin name="box_bot_joint_state" filename="libgazebo_ros_joint_state_publisher.so">
+      <ros>
+          <namespace>/${robot_name}</namespace>
+          <remapping>~/out:=joint_states</remapping>
+      </ros>
+      <update_rate>30</update_rate>
+      <joint_name>joint_left_wheel</joint_name>
+      <joint_name>joint_right_wheel</joint_name>
+      <joint_name>front_yaw_joint</joint_name>
+      <joint_name>back_yaw_joint</joint_name>
+      <joint_name>front_roll_joint</joint_name>
+      <joint_name>back_roll_joint</joint_name>
+      <joint_name>front_pitch_joint</joint_name>
+      <joint_name>back_pitch_joint</joint_name>
+    </plugin>
+  </gazebo>
+  <gazebo>
+    <plugin filename="libgazebo_ros_diff_drive.so" name="differential_drive_controller">
+        <ros>
+            <namespace>/${robot_name}</namespace>
+            <remapping>/cmd_vel:=cmd_vel</remapping>
+        </ros>
+        <update_rate>100</update_rate>
+        <!-- Wheel joints -->
+        <left_joint>joint_left_wheel</left_joint>
+        <right_joint>joint_right_wheel</right_joint>
+        <!-- Kinematics -->
+        <wheel_separation>0.1</wheel_separation>
+        <wheel_diameter>0.07</wheel_diameter>
+        <publish_odom>true</publish_odom>
+        <!-- TF frames -->
+        <odometry_frame>${robot_name}/odom</odometry_frame>>
+        <robot_base_frame>${robot_name}/base_link</robot_base_frame>
+        <publish_odom_tf>true</publish_odom_tf>
+        <publish_wheel_tf>false</publish_wheel_tf>
+        <!-- Limits -->
+        <max_wheel_torque>1.0</max_wheel_torque>
+        <max_wheel_acceleration>2.0</max_wheel_acceleration>
+    </plugin>
+  </gazebo>
 </robot>
